File: tvp_board.sch (KiCad schematic (older format))
At the start: 87 parts, among them J1 VGA, J2 3XRCA_CONN, J3 SCART-F, J5 5VDC_IN, J6 SJ1-3533NG, J7 SJ1-3533NG, SW1 SPST, SW4 DPDT, U1 TVP7002PZP, U17 THS7353, U4 SN74LVC2G17, U5 AP7361C, U6 TLV70033, U7 NCP703SN19T1G, U9 TLV70019, Y1 ACHL-27MHZ-EK

Commit message: add test pins fix tracks
Connections:
- wire segments 237 -> 273
Changed lines of the file:
@@
 EESchema Schematic File Version 4
 LIBS:ossc_board-cache
-EELAYER 26 0
+EELAYER 30 0
 EELAYER END
 $Descr A4 11693 8268
@@
 	10850 6250 10850 6300
 Wire Wire Line
-	9700 6250 10850 6250
-Wire Wire Line
-	9550 6550 9850 6550
-Wire Wire Line
-	9350 3450 9350 6100
+	9700 6250 10300 6250
+Wire Wire Line
+	9550 6550 9700 6550
+Wire Wire Line
+	9350 3450 9350 3900
 Wire Wire Line
 	4850 7100 4700 7100
@@
 Connection ~ 3500 3100
 Wire Wire Line
-	3500 3200 3500 2900
+	3500 3200 3500 3100
 Wire Wire Line
 	3500 2900 3700 2900
@@
 	10300 6250 10300 6200
 Wire Wire Line
-	7800 6100 8350 6100
+	7800 6100 8100 6100
 Connection ~ 8100 6100
 Wire Wire Line
@@
 	4600 2100 4600 2050
 Wire Wire Line
-	3550 7000 4400 7000
-Wire Wire Line
-	3550 7100 4400 7100
+	3550 7000 4250 7000
+Wire Wire Line
+	3550 7100 4250 7100
 Wire Wire Line
 	2650 2600 3400 2600
 Connection ~ 3600 7200
 Wire Wire Line
-	3550 7200 3800 7200
+	3550 7200 3600 7200
 Connection ~ 850  6600
 Wire Wire Line
-	700  6600 1650 6600
+	700  6600 850  6600
 Wire Wire Line
 	3450 2700 3700 2700
@@
 	3700 4100 3200 4100
 Wire Wire Line
-	3550 6800 4000 6800
-Wire Wire Line
-	3550 6600 4000 6600
-Wire Wire Line
-	3550 6400 4000 6400
+	3550 6800 3600 6800
+Wire Wire Line
+	3550 6600 3600 6600
+Wire Wire Line
+	3550 6400 3600 6400
 Wire Wire Line
 	700  6600 700  6250
@@
 	7050 7050 7300 7050
 Wire Wire Line
-	7050 6950 7450 6950
+	7050 6950 7100 6950
 Wire Wire Line
 	6600 1750 6600 2100
@@
 	6300 1450 6300 1550
 Wire Wire Line
-	6100 1450 6300 1450
+	6100 1450 6200 1450
 Wire Wire Line
 	6500 1750 6500 2100
 Wire Wire Line
-	8750 950  9250 950
+	8750 950  9100 950
 Wire Wire Line
 	9100 850  8750 850
 Connection ~ 6200 1450
 Wire Wire Line
-	6200 1450 6200 2100
+	6200 1450 6200 1600
 Wire Wire Line
 	6100 1450 6100 2100
@@
 	5700 1350 5800 1350
 Wire Wire Line
-	5700 1000 5700 2100
+	5700 1000 5700 1350
 Wire Wire Line
 	5800 2100 5800 1750
@@
 	5300 1950 5300 2100
 Wire Wire Line
-	5200 1950 5500 1950
+	5200 1950 5300 1950
 Wire Wire Line
 	5200 2100 5200 1950
@@
 	5000 1800 5000 2100
 Wire Wire Line
-	4800 1100 4800 800
+	4800 1100 4800 1050
 Wire Wire Line
 	4800 1400 4800 2100
 Wire Wire Line
-	2450 3000 3500 3000
+	2450 3000 3350 3000
 Wire Wire Line
 	3500 3200 3700 3200
@@
 Wire Wire Line
 	550  5550 850  5550
-Connection ~ 9350 6100
 Connection ~ 9700 5850
 Connection ~ 9700 6550
@@
 	7600 6200 7600 6300
 Wire Wire Line
-	7600 6300 7800 6300
+	7600 6300 7650 6300
 Connection ~ 10850 6550
 Wire Wire Line
@@
 	10300 6900 10300 6950
 Wire Wire Line
-	9700 6950 10850 6950
-Wire Wire Line
-	10750 5850 11050 5850
-Wire Wire Line
-	10750 6550 11050 6550
+	9700 6950 10300 6950
+Wire Wire Line
+	10750 5850 10850 5850
+Wire Wire Line
+	10750 6550 10850 6550
 Wire Wire Line
 	9850 6550 9850 6700
@@
 	10250 4900 10250 4950
 Wire Wire Line
-	9650 4950 10800 4950
-Wire Wire Line
-	9350 4550 9800 4550
-Wire Wire Line
-	10700 4550 11000 4550
+	9650 4950 10250 4950
+Wire Wire Line
+	9350 4550 9650 4550
+Wire Wire Line
+	10700 4550 10800 4550
 Wire Wire Line
 	9800 4550 9800 4700
@@
 	10250 4200 10250 4300
 Wire Wire Line
-	9650 4300 10800 4300
-Wire Wire Line
-	9350 3900 9850 3900
-Wire Wire Line
-	10650 3900 11000 3900
+	9650 4300 10250 4300
+Wire Wire Line
+	9350 3900 9650 3900
+Wire Wire Line
+	10650 3900 10800 3900
 Wire Wire Line
 	11000 3900 11000 3950
@@
 Connection ~ 6950 1050
 Wire Wire Line
-	9550 5500 9550 6550
+	9550 5500 9550 5850
 Connection ~ 9550 5850
 Wire Wire Line
-	9850 5850 9550 5850
+	9850 5850 9700 5850
 Wire Wire Line
 	10050 5500 9550 5500
@@
 Wire Wire Line
 	3950 5900 3750 5900
+Wire Wire Line
+	4250 7000 4400 7000
+Wire Wire Line
+	4250 7100 4400 7100
+Wire Wire Line
+	6200 1600 6200 2100
+Wire Wire Line
+	3350 3000 3500 3000
+Wire Wire Line
+	3500 3000 3500 2900
+Wire Wire Line
+	3500 3100 3500 3000
+Wire Wire Line
+	10300 6250 10850 6250
+Wire Wire Line
+	8100 6100 8350 6100
+Wire Wire Line
+	3600 7200 3800 7200
+Wire Wire Line
+	850  6600 1650 6600
+Wire Wire Line
+	3600 6800 4000 6800
+Wire Wire Line
+	3600 6600 4000 6600
+Wire Wire Line
+	3600 6400 4000 6400
+Wire Wire Line
+	9100 950  9250 950
+Wire Wire Line
+	6200 1450 6300 1450
+Wire Wire Line
+	5700 1350 5700 2100
+Wire Wire Line
+	5300 1950 5500 1950
+Wire Wire Line
+	9700 5850 9550 5850
+Wire Wire Line
+	9700 6550 9850 6550
+Wire Wire Line
+	10850 6550 11050 6550
+Wire Wire Line
+	10300 6950 10850 6950
+Wire Wire Line
+	7650 6300 7800 6300
+Wire Wire Line
+	9650 4550 9800 4550
+Wire Wire Line
+	10800 4550 11000 4550
+Wire Wire Line
+	10250 4950 10800 4950
+Wire Wire Line
+	9650 3900 9850 3900
+Wire Wire Line
+	10800 3900 11000 3900
+Wire Wire Line
+	10250 4300 10800 4300
+Wire Wire Line
+	9350 4550 9350 5600
+Wire Wire Line
+	9350 3900 9350 4550
+Wire Wire Line
+	7350 6950 7450 6950
+Wire Wire Line
+	7100 6950 7350 6950
+Wire Wire Line
+	9350 5600 9350 6100
+Wire Wire Line
+	9550 5850 9550 6550
+Wire Wire Line
+	10850 5850 11050 5850
+Wire Wire Line
+	4800 1050 4800 800
 $EndSCHEMATC

Commit message: remove unnecessary component
Parts:
- removed C12, C3, C4, C5, C6, C7: 1u, custom_components:SM0603_Capa_libcms, symbol ossc_board-rescue:C
- removed C33, C36: 22p, custom_components:SM0603_Capa_libcms, symbol ossc_board-rescue:C
- removed C70: 10n, custom_components:SM0603_Capa_libcms, symbol ossc_board-rescue:C-RESCUE-ossc_board
- removed C71: 47u, custom_components:SM0805_libcms, symbol ossc_board-rescue:C-RESCUE-ossc_board
- removed J2: 3XRCA_CONN, custom_components:3xRCA_CONN, symbol ossc_board-rescue:3xRCA_CONN
- removed J3: SCART-F, custom_components:SCART_CONN, symbol ossc_board-rescue:SCART-F
- removed J6, J7: SJ1-3533NG, custom_components:SJ1-3533NG, symbol ossc_board-rescue:CONN_01X03
- removed R38, R44: 100, custom_components:SM0603_Resistor_libcms, symbol ossc_board-rescue:R
- removed R4, R5, R6, R7, R8, R9: 75, custom_components:SM0603_Resistor_libcms, symbol ossc_board-rescue:R
- removed SW4: DPDT, custom_components:MS22, symbol ossc_board-rescue:DPDT
- removed U17: THS7353, custom_components:TSSOP-20_4.4x6.5mm_Pitch0.65mm_Handsoldering, symbol ossc_board-rescue:THS7353
- added C33: 1u, custom_components:SM0603_Capa_libcms, symbol ossc_board-rescue:C-RESCUE-ossc_board
- C100, C103, C76: value 0.1u -> 10n
- C11: value 1n -> 10n
Connections:
- net labels removed: AV1_AUD_L, AV1_AUD_R, AV2_AUD_L, AV2_AUD_R, AV3_AUD_L, AV3_AUD_R, RGB1_B, RGB1_G, RGB1_R, RGB2_B, RGB2_G, RGB2_R, RGB_12_B, RGB_12_G, RGB_12_R
- wire segments 273 -> 208
- no-connect marks 22 -> 13
Other:
- note removed: "max. 25mA"

Commit message: update PCB
Parts:
- removed D5: SD05-7, custom_components:SOD-323_Handsoldering, symbol ossc_board-rescue:ZENER
- removed J1: VGA, custom_components:VGA_CONN, symbol ossc_board-rescue:VGA
- removed J5: 5VDC_IN, custom_components:BARREL_JACK_roundconn, symbol ossc_board-rescue:BARREL_JACK
- removed SW1: SPST, custom_components:SW_SPDT, symbol ossc_board-rescue:SPST
- C1, C10, C100, C103, C104, C105, C106, C109, C11, C13, C14, C15, C16, C17, C18, C19, C2, C20, C21, C22, C23, C24, C25, C26, C27, C28, C31, C32, C33, C34, C35, C37, C38, C72, C76, C8, C9, C93, C95: footprint custom_components:SM0603_Capa_libcms -> Capacitor_SMD:C_0603_1608Metric_Pad1.05x0.95mm_HandSolder
- C107: footprint custom_components:SM0805_libcms -> Capacitor_SMD:C_0805_2012Metric_Pad1.15x1.40mm_HandSolder
- F4: renamed from F1; footprint custom_components:SM0603_Resistor_libcms -> Inductor_SMD:L_0603_1608Metric_Pad1.05x0.95mm_HandSolder
- FB5, FB6, FB7: footprint custom_components:SM0603_Resistor_libcms -> Inductor_SMD:L_0603_1608Metric_Pad1.05x0.95mm_HandSolder
- R1, R10, R11, R12, R13, R14, R15, R2, R3: footprint custom_components:SM0603_Resistor_libcms -> Resistor_SMD:R_0603_1608Metric_Pad1.05x0.95mm_HandSolder
Connections:
- net labels added: 5VDC_IN
- net labels removed: RGB1_S
- wire segments 208 -> 196
- no-connect marks 13 -> 8
Other:
- moved on the sheet: F4

Commit message: update PCB 2
Changed lines of the file:
@@
 Text Label 10950 6550 0    60   ~ 0
 DVDD
-Text Label 2100 1350 0    60   ~ 0
+Text Label 2350 5850 0    60   ~ 0
 RGB3_HS
-Text Label 2100 1150 0    60   ~ 0
+Text Label 2350 5650 0    60   ~ 0
 RGB3_VS
 $Comp
@@
 	7450 6700 7550 6700
 Connection ~ 7450 6950
-Text HLabel 3000 1150 2    60   Input ~ 0
+Text HLabel 3250 5650 2    60   Input ~ 0
 RGB3_VS
-Text HLabel 3000 1350 2    60   Input ~ 0
+Text HLabel 3250 5850 2    60   Input ~ 0
 RGB3_HS
 Wire Wire Line
-	2100 1150 3000 1150
-Wire Wire Line
-	2100 1350 3000 1350
+	2350 5650 3250 5650
+Wire Wire Line
+	2350 5850 3250 5850
 Text HLabel 4800 800  2    60   Input ~ 0
 RGB3_G

Commit message: update3
Parts:
- removed F4: F0603E1R50FSTR, Inductor_SMD:L_0603_1608Metric_Pad1.05x0.95mm_HandSolder, symbol ossc_board-rescue:F_Small
Changed lines of the file:
@@
-$EndComp
-$Comp
-L ossc_board-rescue:F_Small F4
-U 1 1 55ECFDAC
-P 8800 6700
-F 0 "F4" H 8760 6760 50  0000 L CNN
-F 1 "F0603E1R50FSTR" H 8750 6850 50  0000 L CNN
-F 2 "Inductor_SMD:L_0603_1608Metric_Pad1.05x0.95mm_HandSolder" H 8800 6700 60  0001 C CNN
-F 3 "" H 8800 6700 60  0000 C CNN
-	1    8800 6700
-	1    0    0    -1
 $EndComp
 $Comp

Commit message: minor update
Parts:
- removed C107: 47u, Capacitor_SMD:C_0805_2012Metric_Pad1.15x1.40mm_HandSolder, symbol ossc_board-rescue:C-RESCUE-ossc_board
Connections:
- wire segments 196 -> 194
Changed lines of the file:
@@
 Text Label 9450 2750 0    60   ~ 0
 RESET_N
-$Comp
-L ossc_board-rescue:PWR_FLAG #FLG0131
-U 1 1 54049F52
-P 9350 5600
-F 0 "#FLG0131" H 9350 5695 30  0001 C CNN
-F 1 "PWR_FLAG" H 9350 5780 30  0000 C CNN
-F 2 "" H 9350 5600 60  0001 C CNN
-F 3 "" H 9350 5600 60  0000 C CNN
-	1    9350 5600
-	0    -1   -1   0
-$EndComp
 NoConn ~ 5700 5500
 NoConn ~ 5800 5500
@@
 $EndComp
 $Comp
-L ossc_board-rescue:C-RESCUE-ossc_board C107
-U 1 1 55EC52FF
-P 8350 6300
-F 0 "C107" H 8350 6400 40  0000 L CNN
-F 1 "47u" H 8356 6215 40  0000 L CNN
-F 2 "Capacitor_SMD:C_0805_2012Metric_Pad1.15x1.40mm_HandSolder" H 8388 6150 30  0001 C CNN
-F 3 "~" H 8350 6300 60  0000 C CNN
-	1    8350 6300
-	1    0    0    -1
-$EndComp
-$Comp
-L ossc_board-rescue:GND-RESCUE-ossc_board #PWR0150
-U 1 1 55EC5BFD
-P 8350 6500
-F 0 "#PWR0150" H 8350 6500 30  0001 C CNN
-F 1 "GND" H 8350 6430 30  0001 C CNN
-F 2 "" H 8350 6500 60  0001 C CNN
-F 3 "" H 8350 6500 60  0000 C CNN
-	1    8350 6500
-	1    0    0    -1
-$EndComp
-$Comp
 L ossc_board-rescue:FILTER FB6
 U 1 1 55F21890
@@
 	8350 6950 8150 6950
 Connection ~ 7100 6950
-Connection ~ 9350 5600
 Wire Wire Line
 	9450 3200 9900 3200
@@
 	10250 4300 10800 4300
 Wire Wire Line
-	9350 4550 9350 5600
-Wire Wire Line
 	9350 3900 9350 4550
 Wire Wire Line
@@
 Wire Wire Line
 	7100 6950 7350 6950
-Wire Wire Line
-	9350 5600 9350 6100
 Wire Wire Line
 	9550 5850 9550 6550
@@
 Text HLabel 2500 4100 0    60   Input ~ 0
 RGB3_B
-Wire Wire Line
-	9350 6100 8350 6100
-Connection ~ 8350 6100
 Text HLabel 7800 6100 0    60   Input ~ 0
 5VDC_IN
 Wire Wire Line
-	7800 6100 8350 6100
+	7800 6100 9350 6100
+Wire Wire Line
+	9350 4550 9350 6100
 $EndSCHEMATC

Commit message: add dxf update pcb
Parts:
- removed R3: 75, Resistor_SMD:R_0603_1608Metric_Pad1.05x0.95mm_HandSolder, symbol ossc_board-rescue:R
- C100, C103, C104, C105, C106, C11, C17, C25, C76: value 10n -> 0.01u
- C13, C16: value 1n -> 1000p
- C19: value 4.7n -> 4700p
- R15: value 2.2k -> 10k
Changed lines of the file:
@@
 $EndComp
 $Comp
-L ossc_board-rescue:TLV71209DBV-RESCUE-ossc_board U9
+L ossc_board-rescue:TLV71209DBV-RESCUE-ossc_board U?
 U 1 1 53FA4F27
 P 10300 6600
-AR Path="/53FA4F27" Ref="U9"  Part="1"
+AR Path="/53FA4F27" Ref="U?"  Part="1"
 AR Path="/54FDD796/53FA4F27" Ref="U9"  Part="1"
 F 0 "U9" H 10050 6800 40  0000 C CNN
@@
 P 3550 2600
 F 0 "C11" H 3550 2700 40  0000 L CNN
-F 1 "10n" H 3556 2515 40  0000 L CNN
+F 1 "0.01u" H 3556 2515 40  0000 L CNN
 F 2 "Capacitor_SMD:C_0603_1608Metric_Pad1.05x0.95mm_HandSolder" H 3588 2450 30  0001 C CNN
 F 3 "~" H 3550 2600 60  0000 C CNN
@@
 P 4700 1900
 F 0 "C13" H 4700 2000 40  0000 L CNN
-F 1 "1n" H 4706 1815 40  0000 L CNN
+F 1 "1000p" H 4706 1815 40  0000 L CNN
 F 2 "Capacitor_SMD:C_0603_1608Metric_Pad1.05x0.95mm_HandSolder" H 4738 1750 30  0001 C CNN
 F 3 "~" H 4700 1900 60  0000 C CNN
@@
 P 4900 1900
 F 0 "C16" H 4900 2000 40  0000 L CNN
-F 1 "1n" H 4906 1815 40  0000 L CNN
+F 1 "1000p" H 4906 1815 40  0000 L CNN
 F 2 "Capacitor_SMD:C_0603_1608Metric_Pad1.05x0.95mm_HandSolder" H 4938 1750 30  0001 C CNN
 F 3 "~" H 4900 1900 60  0000 C CNN
@@
 P 5000 1600
 F 0 "C17" H 5000 1700 40  0000 L CNN
-F 1 "10n" H 5006 1515 40  0000 L CNN
+F 1 "0.01u" H 5006 1515 40  0000 L CNN
 F 2 "Capacitor_SMD:C_0603_1608Metric_Pad1.05x0.95mm_HandSolder" H 5038 1450 30  0001 C CNN
 F 3 "~" H 5000 1600 60  0000 C CNN
@@
 P 5800 1550
 F 0 "C19" H 5800 1650 40  0000 L CNN
-F 1 "4.7n" H 5806 1465 40  0000 L CNN
+F 1 "4700p" H 5806 1465 40  0000 L CNN
 F 2 "Capacitor_SMD:C_0603_1608Metric_Pad1.05x0.95mm_HandSolder" H 5838 1400 30  0001 C CNN
 F 3 "~" H 5800 1550 60  0000 C CNN
@@
 CLK27
 $Comp
-L ossc_board-rescue:ACHL-27MHZ-EK Y1
+L ossc_board-rescue:ACHL-27MHZ-EK Y?
 U 1 1 53FD28BE
 P 6100 7000
-AR Path="/53FD28BE" Ref="Y1"  Part="1"
+AR Path="/53FD28BE" Ref="Y?"  Part="1"
 AR Path="/54FDD796/53FD28BE" Ref="Y1"  Part="1"
 F 0 "Y1" H 6100 6900 50  0000 C CNN
@@
 P 7350 6750
 F 0 "C25" H 7350 6850 40  0000 L CNN
-F 1 "10n" H 7356 6665 40  0000 L CNN
+F 1 "0.01u" H 7356 6665 40  0000 L CNN
 F 2 "Capacitor_SMD:C_0603_1608Metric_Pad1.05x0.95mm_HandSolder" H 7388 6600 30  0001 C CNN
 F 3 "~" H 7350 6750 60  0000 C CNN
@@
 F 3 "" H 8500 3500 60  0000 C CNN
 	1    8500 3500
-	0    -1   -1   0
-$EndComp
-$Comp
-L ossc_board-rescue:R-RESCUE-ossc_board R15
-U 1 1 53FD2FC9
-P 8450 3000
-F 0 "R15" V 8530 3000 40  0000 C CNN
-F 1 "2.2k" V 8457 3001 40  0000 C CNN
-F 2 "Resistor_SMD:R_0603_1608Metric_Pad1.05x0.95mm_HandSolder" V 8380 3000 30  0001 C CNN
-F 3 "~" H 8450 3000 30  0000 C CNN
-	1    8450 3000
 	0    -1   -1   0
 $EndComp
@@
 max. 20mA
 $Comp
-L ossc_board-rescue:TLV71209DBV-RESCUE-ossc_board U6
+L ossc_board-rescue:TLV71209DBV-RESCUE-ossc_board U?
 U 1 1 5509C1FA
 P 10250 4600
-AR Path="/5509C1FA" Ref="U6"  Part="1"
+AR Path="/5509C1FA" Ref="U?"  Part="1"
 AR Path="/54FDD796/5509C1FA" Ref="U6"  Part="1"
 F 0 "U6" H 10000 4800 40  0000 C CNN
@@
 $EndComp
 $Comp
-L ossc_board-rescue:TLV71209DBV-RESCUE-ossc_board U7
+L ossc_board-rescue:TLV71209DBV-RESCUE-ossc_board U?
 U 1 1 5511AE30
 P 10300 5900
-AR Path="/5511AE30" Ref="U7"  Part="1"
+AR Path="/5511AE30" Ref="U?"  Part="1"
 AR Path="/54FDD796/5511AE30" Ref="U7"  Part="1"
 F 0 "U7" H 10050 6100 40  0000 C CNN
@@
 Text Label 9350 5500 1    60   ~ 0
 5VDC
-$Comp
-L ossc_board-rescue:R R3
-U 1 1 55C155CD
-P 4250 1750
-F 0 "R3" V 4330 1750 40  0000 C CNN
-F 1 "75" V 4257 1751 40  0000 C CNN
-F 2 "Resistor_SMD:R_0603_1608Metric_Pad1.05x0.95mm_HandSolder" V 4180 1750 30  0001 C CNN
-F 3 "~" H 4250 1750 30  0000 C CNN
-	1    4250 1750
-	1    0    0    -1
-$EndComp
 $Comp
 L ossc_board-rescue:GND-RESCUE-ossc_board #PWR0136
@@
 P 3300 2700
 F 0 "C103" H 3300 2800 40  0000 L CNN
-F 1 "10n" H 3306 2615 40  0000 L CNN
+F 1 "0.01u" H 3306 2615 40  0000 L CNN
 F 2 "Capacitor_SMD:C_0603_1608Metric_Pad1.05x0.95mm_HandSolder" H 3338 2550 30  0001 C CNN
 F 3 "~" H 3300 2700 60  0000 C CNN
@@
 P 3250 3600
 F 0 "C76" H 3250 3700 40  0000 L CNN
-F 1 "10n" H 3256 3515 40  0000 L CNN
+F 1 "0.01u" H 3256 3515 40  0000 L CNN
 F 2 "Capacitor_SMD:C_0603_1608Metric_Pad1.05x0.95mm_HandSolder" H 3288 3450 30  0001 C CNN
 F 3 "~" H 3250 3600 60  0000 C CNN
@@
 P 3250 4300
 F 0 "C100" H 3250 4400 40  0000 L CNN
-F 1 "10n" H 3256 4215 40  0000 L CNN
+F 1 "0.01u" H 3256 4215 40  0000 L CNN
 F 2 "Capacitor_SMD:C_0603_1608Metric_Pad1.05x0.95mm_HandSolder" H 3288 4150 30  0001 C CNN
 F 3 "~" H 3250 4300 60  0000 C CNN
@@
 P 3550 3500
 F 0 "C104" H 3550 3600 40  0000 L CNN
-F 1 "10n" H 3556 3415 40  0000 L CNN
+F 1 "0.01u" H 3556 3415 40  0000 L CNN
 F 2 "Capacitor_SMD:C_0603_1608Metric_Pad1.05x0.95mm_HandSolder" H 3588 3350 30  0001 C CNN
 F 3 "~" H 3550 3500 60  0000 C CNN
@@
 P 3550 4200
 F 0 "C105" H 3550 4300 40  0000 L CNN
-F 1 "10n" H 3556 4115 40  0000 L CNN
+F 1 "0.01u" H 3556 4115 40  0000 L CNN
 F 2 "Capacitor_SMD:C_0603_1608Metric_Pad1.05x0.95mm_HandSolder" H 3588 4050 30  0001 C CNN
 F 3 "~" H 3550 4200 60  0000 C CNN
@@
 P 4500 1900
 F 0 "C106" H 4500 2000 40  0000 L CNN
-F 1 "10n" H 4506 1815 40  0000 L CNN
+F 1 "0.01u" H 4506 1815 40  0000 L CNN
 F 2 "Capacitor_SMD:C_0603_1608Metric_Pad1.05x0.95mm_HandSolder" H 4538 1750 30  0001 C CNN
 F 3 "~" H 4500 1900 60  0000 C CNN
@@
 	1    3350 3000
 	1    0    0    -1
-$EndComp
-$Comp
-L ossc_board-rescue:GND-RESCUE-ossc_board #PWR0155
-U 1 1 55F350C7
-P 8700 3000
-F 0 "#PWR0155" H 8700 3000 30  0001 C CNN
-F 1 "GND" H 8700 2930 30  0001 C CNN
-F 2 "" H 8700 3000 60  0001 C CNN
-F 3 "" H 8700 3000 60  0000 C CNN
-	1    8700 3000
-	0    -1   -1   0
 $EndComp
 Text Label 2750 3000 0    60   ~ 0
@@
 	4250 1450 4700 1450
 Wire Wire Line
-	4250 1600 4250 1450
-Wire Wire Line
 	7050 850  6600 850
 Wire Wire Line
@@
 Wire Wire Line
 	9350 4550 9350 6100
+Wire Wire Line
+	4250 1450 4250 1900
+$Comp
+L ossc_board-rescue:R-RESCUE-ossc_board R15
+U 1 1 53FD2FC9
+P 8450 3000
+F 0 "R15" V 8530 3000 40  0000 C CNN
+F 1 "10k" V 8457 3001 40  0000 C CNN
+F 2 "Resistor_SMD:R_0603_1608Metric_Pad1.05x0.95mm_HandSolder" V 8380 3000 30  0001 C CNN
+F 3 "~" H 8450 3000 30  0000 C CNN
+	1    8450 3000
+	0    -1   -1   0
+$EndComp
+$Comp
+L ossc_board-rescue:GND-RESCUE-ossc_board #PWR0155
+U 1 1 55F350C7
+P 8700 3000
+F 0 "#PWR0155" H 8700 3000 30  0001 C CNN
+F 1 "GND" H 8700 2930 30  0001 C CNN
+F 2 "" H 8700 3000 60  0001 C CNN
+F 3 "" H 8700 3000 60  0000 C CNN
+	1    8700 3000
+	0    -1   -1   0
+$EndComp
 $EndSCHEMATC
