File: soundbox.sch (KiCad schematic (older format))
At the start: 179 parts, among them J10 COLOR INPUT, J11 MONO INPUT, J12 NEXT PWR INPUT 1, J13 NEXT PWR INPUT 2, J14 -12VDC OUT, J15 5VDC STANDBY, J16 MON IN 1, J17 MON IN 2, J18 PA1, J19 BOOT0, J2 OUT (SJ1-3535NG), J20 PC0, J21 PC1, J22 PB0, J23 PB1, J24 R SPK, J25 R SPEAKER (SJ-2509N), J26 L SPEAKER, J27 L SPK, J28 I2C Ext, J29 OLED, J3 MIC (SJ1-3535NG), J31 NeXT Keyboard, J32 NeXT Keyboard (MD-50SM / KMDG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, J4 USB Host (SS-52100-001), J5 Mic IN, J6 Audio OUT, J7 STLINK, J8 UART2, J9 PA0, Q1 2SC2712, SW1 NeXT POWER SW (1-1825027-1 / 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, SW3 NeXT POWER SW, SW4 MCU RESET, U11 TLV70033DDCR, U17 USBLC6-2SC6, U18 STMPS2141STR, U19 SN74LVC2G34DBV, U20 PCM5122PW, U21 TLV70033DDCR (or XC6204B332MR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, U22 TLV70033DDCR (or XC6204B332MR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, U23 PLT133/T, U24 STM32F401RCT6, U25 SN74LVC1G07DBV, U26 SN74HCT125DR, U27 TLV320ADC3100, U28 BD33FC0FP, U29 TPA2005D1DGN, U30 BD33FC0FP, U31 TPA2005D1DGN, U32 PCA9515D, U8 5V(DC/DC), X3 ECS-2520MVLC-225.792-BN-TR, Y2 25MHz (FA-238 25.0000MB-K0)

Commit message: minor update
Parts:
- added D9: (RB160M-30TR), custom_components:D_SOD-123_HandSoldering, symbol Device:D_ALT
Connections:
- net 5VDC_OUT: now also D9.2 (A)
- net at C30.1, C5.2, D5.1 (K)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: now also D9.1 (K)
Changed lines of the file:
@@
 Wire Wire Line
 	4250 2950 4250 3100
-$Comp
-L Connector_Generic:Conn_01x02 JP1
-U 1 1 5F692B96
-P 5250 2500
-F 0 "JP1" H 5330 2492 50  0000 L CNN
-F 1 "Standby DC From NeXT Hardware" H 5330 2401 50  0000 L CNN
-F 2 "Connector_PinHeader_2.54mm:PinHeader_1x02_P2.54mm_Vertical" H 5250 2500 50  0001 C CNN
-F 3 "~" H 5250 2500 50  0001 C CNN
-	1    5250 2500
-	1    0    0    -1
-$EndComp
 Wire Wire Line
 	3200 2600 3200 2950
@@
 Connection ~ 4900 1750
 Wire Wire Line
-	4900 1750 5050 1750
-Wire Wire Line
-	5050 2500 5050 1750
-Connection ~ 5050 1750
-Wire Wire Line
-	5050 1750 5150 1750
-Wire Wire Line
 	4900 2150 4900 2300
 Wire Wire Line
@@
 Wire Wire Line
 	3450 1750 3750 1750
-Wire Wire Line
-	3750 1750 3750 1850
 Connection ~ 3750 1750
 Wire Wire Line
@@
 Connection ~ 3750 2300
 Connection ~ 3450 2300
-Wire Wire Line
-	3200 2600 5050 2600
 Text Label 2300 1100 0    60   ~ 0
 MONO_VIDEO
@@
 Wire Wire Line
 	6500 4150 6100 4150
-$Comp
-L Jumper:Jumper_3_Open JP2
-U 1 1 5F3E34A1
-P 3200 4950
-F 0 "JP2" H 3200 5174 50  0000 C CNN
-F 1 "KBD_SW" H 3200 5083 50  0000 C CNN
-F 2 "Jumper:SolderJumper-3_P1.3mm_Open_RoundedPad1.0x1.5mm_NumberLabels" H 3200 4950 50  0001 C CNN
-F 3 "~" H 3200 4950 50  0001 C CNN
-	1    3200 4950
-	1    0    0    -1
-$EndComp
-$Comp
-L Jumper:Jumper_3_Open JP3
-U 1 1 5F3F90B6
-P 3200 5300
-F 0 "JP3" H 3200 5524 50  0000 C CNN
-F 1 "KBD_SW" H 3200 5433 50  0000 C CNN
-F 2 "Jumper:SolderJumper-3_P1.3mm_Open_RoundedPad1.0x1.5mm_NumberLabels" H 3200 5300 50  0001 C CNN
-F 3 "~" H 3200 5300 50  0001 C CNN
-	1    3200 5300
-	1    0    0    -1
-$EndComp
-$Comp
-L Jumper:Jumper_3_Open JP4
-U 1 1 5F3F9CBB
-P 3200 5900
-F 0 "JP4" H 3200 6124 50  0000 C CNN
-F 1 "KBD_SW" H 3200 6033 50  0000 C CNN
-F 2 "Jumper:SolderJumper-3_P1.3mm_Open_RoundedPad1.0x1.5mm_NumberLabels" H 3200 5900 50  0001 C CNN
-F 3 "~" H 3200 5900 50  0001 C CNN
-	1    3200 5900
-	1    0    0    -1
-$EndComp
 Wire Wire Line
 	2200 5050 2300 5050
@@
 Wire Wire Line
 	9250 7850 8750 7850
+Wire Wire Line
+	3750 1750 3750 1850
+Wire Wire Line
+	4000 1350 3750 1350
+Wire Wire Line
+	3750 1350 3750 1750
+Wire Wire Line
+	4300 1350 4550 1350
+Wire Wire Line
+	4550 1350 4550 1750
+$Comp
+L Jumper:Jumper_3_Open JP4
+U 1 1 5F3F9CBB
+P 3200 5900
+F 0 "JP4" H 3200 6124 50  0000 C CNN
+F 1 "KBD_SW" H 3200 6033 50  0000 C CNN
+F 2 "Jumper:SolderJumper-3_P1.3mm_Open_RoundedPad1.0x1.5mm_NumberLabels" H 3200 5900 50  0001 C CNN
+F 3 "~" H 3200 5900 50  0001 C CNN
+	1    3200 5900
+	1    0    0    -1
+$EndComp
+$Comp
+L Jumper:Jumper_3_Open JP3
+U 1 1 5F3F90B6
+P 3200 5300
+F 0 "JP3" H 3200 5524 50  0000 C CNN
+F 1 "KBD_SW" H 3200 5433 50  0000 C CNN
+F 2 "Jumper:SolderJumper-3_P1.3mm_Open_RoundedPad1.0x1.5mm_NumberLabels" H 3200 5300 50  0001 C CNN
+F 3 "~" H 3200 5300 50  0001 C CNN
+	1    3200 5300
+	1    0    0    -1
+$EndComp
+$Comp
+L Jumper:Jumper_3_Open JP2
+U 1 1 5F3E34A1
+P 3200 4950
+F 0 "JP2" H 3200 5174 50  0000 C CNN
+F 1 "KBD_SW" H 3200 5083 50  0000 C CNN
+F 2 "Jumper:SolderJumper-3_P1.3mm_Open_RoundedPad1.0x1.5mm_NumberLabels" H 3200 4950 50  0001 C CNN
+F 3 "~" H 3200 4950 50  0001 C CNN
+	1    3200 4950
+	1    0    0    -1
+$EndComp
+$Comp
+L Device:D_ALT D9
+U 1 1 5F5B0860
+P 4150 1350
+F 0 "D9" V 4104 1429 50  0000 L CNN
+F 1 "(RB160M-30TR)" V 4250 1400 50  0000 L CNN
+F 2 "custom_components:D_SOD-123_HandSoldering" H 4150 1350 50  0001 C CNN
+F 3 "~" H 4150 1350 50  0001 C CNN
+	1    4150 1350
+	1    0    0    -1
+$EndComp
+Wire Wire Line
+	5050 1750 5150 1750
+Wire Wire Line
+	4900 1750 5050 1750
+Connection ~ 5050 1750
+Wire Wire Line
+	5050 2500 5050 1750
+Wire Wire Line
+	3200 2600 5050 2600
+$Comp
+L Connector_Generic:Conn_01x02 JP1
+U 1 1 5F692B96
+P 5250 2500
+F 0 "JP1" H 5330 2492 50  0000 L CNN
+F 1 "Standby DC From NeXT Hardware" H 5330 2401 50  0000 L CNN
+F 2 "Connector_PinHeader_2.54mm:PinHeader_1x02_P2.54mm_Vertical" H 5250 2500 50  0001 C CNN
+F 3 "~" H 5250 2500 50  0001 C CNN
+	1    5250 2500
+	1    0    0    -1
+$EndComp
 $EndSCHEMATC
