File: soundbox.sch (KiCad schematic (older format))
At the start: 191 parts, among them J10 COLOR INPUT, J11 MONO INPUT, J12 NEXT PWR INPUT 1, J13 NEXT PWR INPUT 2, J14 -12VDC OUT, J15 5VDC STANDBY, J16 MON IN 1, J17 MON IN 2, J18 PA1, J19 BOOT0, J2 OUT (SJ1-3535NG), J20 PC0, J21 PC1, J22 PB0, J23 PB1, J24 R SPK, J25 R SPEAKER (SJ-2509N), J26 L SPEAKER, J27 L SPK, J28 I2C Ext, J29 OLED, J3 MIC (SJ1-3535NG), J30 BOOT1, J31 NeXT Keyboard, J32 NeXT Keyboard (MD-50SM / KMDG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, J4 USB Host (SS-52100-001), J5 Mic IN, J6 Audio OUT, J7 STLINK, J8 UART2, J9 PA0, Q1 2SC2712, SW1 NeXT POWER SW (1-1825027-1 / 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, SW3 NeXT POWER SW, SW4 MCU RESET, U11 TLV70033DDCR, U17 USBLC6-2SC6, U18 STMPS2151STR‎ or TPS2051CDBV, U19 SN74LVC2G34DBV, U20 PCM5122PW, U21 TLV70033DDCR (or XC6204B332MR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, U22 TLV70033DDCR (or XC6204B332MR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, U23 PLT133/T, U24 STM32F401RCT6, U25 SN74LVC1G07DBV, U26 SN74HC125DR, U27 TLV320ADC3100, U28 BD33FC0FP, U29 TPA2005D1DGN, U30 BD33FC0FP, U31 TPA2005D1DGN, U32 (PCA9515AD), U8 5V(DC/DC), X3 ECS-2520MVLC-225.792-BN-TR, Y2 25MHz (FA-238 25.0000MB-K0)

Commit message: add caps
Parts:
- removed J14: -12VDC OUT, Connector_JST:JST_XH_B2B-XH-A_1x02_P2.50mm_Vertical, symbol Connector:Conn_01x02_Male
- removed JP6: Use Dummy Load, Connector_PinHeader_2.54mm:PinHeader_1x02_P2.54mm_Vertical, symbol Connector_Generic:Conn_01x02
- removed R31: 100//100 5W (or 47ohm 7W), Resistor_THT:R_Axial_DIN0617_L17.0mm_D6.0mm_P30.48mm_Horizontal, symbol Device:R
- added C179, C181: 1u, Capacitor_SMD:C_0603_1608Metric_Pad1.08x0.95mm_HandSolder, symbol Device:C
- added C180, C182: 47u, Capacitor_SMD:CP_Elec_5x5.3, symbol Device:CP
- added D12: (RB160M-30TR), custom_components:D_SOD-123_HandSoldering, symbol Device:D_ALT
- added U33: 5V(DC/DC), Package_TO_SOT_THT:TO-220-3_Vertical, symbol Regulator_Linear:L7805
- J12: value NEXT PWR INPUT 1 -> NEXT PWR IN 1
- J13: value NEXT PWR INPUT 2 -> NEXT PWR IN 2
Connections:
- net 5VDC_OUT: no longer JP1.1 (Pin_1)
- net 5VDC_STBY: now also C181.2, C182.1, D12.2 (A), U33.3 (OUT); no longer JP1.2 (Pin_2)
- net GND: now also C179.1, C180.2, C181.1, C182.2, U33.2 (GND)
- net at C30.1, C5.2, D5.1 (K)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: now also JP1.1 (Pin_1)
- net -12V: no longer names the net of J12.3 (Pin_3)
- net -12V: no longer J13.3 (Pin_3)
- new net: C179.2, C180.1, D12.1 (K), JP1.2 (Pin_2), U33.1 (IN)
- no-connect marks 38 -> 40
Other:
- note added: "-12V not used"
- note removed: "-12V Dummy Load for older PSU"
- moved on the sheet: JP1
Changed lines of the file:
@@
 P 1600 1750
 F 0 "J12" H 1708 2031 50  0000 C CNN
-F 1 "NEXT PWR INPUT 1" H 1550 1950 50  0000 C CNN
+F 1 "NEXT PWR IN 1" H 1550 1950 50  0000 C CNN
 F 2 "Connector_JST:JST_XH_B3B-XH-A_1x03_P2.50mm_Vertical" H 1600 1750 50  0001 C CNN
 F 3 "~" H 1600 1750 50  0001 C CNN
@@
 P 2000 1750
 F 0 "J13" H 2108 2031 50  0000 C CNN
-F 1 "NEXT PWR INPUT 2" H 2350 1950 50  0000 C CNN
+F 1 "NEXT PWR IN 2" H 2350 1950 50  0000 C CNN
 F 2 "Connector_JST:JST_XH_B3B-XH-A_1x03_P2.50mm_Vertical" H 2000 1750 50  0001 C CNN
 F 3 "~" H 2000 1750 50  0001 C CNN
@@
 	1800 1750 2200 1750
 Connection ~ 2200 1750
-Wire Wire Line
-	1800 1850 2200 1850
-Wire Wire Line
-	2200 1850 2450 1850
-Connection ~ 2200 1850
 Text Label 2450 1750 0    60   ~ 0
 12V
-Text Label 2450 1850 0    60   ~ 0
--12V
 $Comp
 L Device:Fuse_Small F3
@@
 P 3150 2000
 F 0 "D5" V 3104 2079 50  0000 L CNN
-F 1 "RB160M-30TR" V 3250 2050 50  0000 L CNN
+F 1 "RB160M-30TR" V 3300 1700 50  0000 L CNN
 F 2 "custom_components:D_SOD-123_HandSoldering" H 3150 2000 50  0001 C CNN
 F 3 "~" H 3150 2000 50  0001 C CNN
@@
 Connection ~ 3450 1750
 Wire Wire Line
-	3450 1750 3150 1750
+	3450 1750 3300 1750
 Wire Wire Line
 	4450 1750 4550 1750
@@
 	2200 2950 2850 2950
 $Comp
-L Connector:Conn_01x02_Male J14
-U 1 1 5F68323C
-P 2000 2300
-F 0 "J14" H 1973 2182 50  0000 R CNN
-F 1 "-12VDC OUT" H 1973 2273 50  0000 R CNN
-F 2 "Connector_JST:JST_XH_B2B-XH-A_1x02_P2.50mm_Vertical" H 2000 2300 50  0001 C CNN
-F 3 "~" H 2000 2300 50  0001 C CNN
-	1    2000 2300
-	1    0    0    1
-$EndComp
-$Comp
-L ossc_board-rescue:GND-RESCUE-ossc_board #PWR0151
-U 1 1 5F68409E
-P 2350 2400
-F 0 "#PWR0151" H 2350 2400 30  0001 C CNN
-F 1 "GND-RESCUE-ossc_board" H 2350 2330 30  0001 C CNN
-F 2 "" H 2350 2400 60  0000 C CNN
-F 3 "" H 2350 2400 60  0000 C CNN
-	1    2350 2400
-	1    0    0    -1
-$EndComp
-Wire Wire Line
-	2200 2300 2350 2300
-Wire Wire Line
-	2350 2300 2350 2400
-Wire Wire Line
-	2200 2200 2450 2200
-Wire Wire Line
-	2450 2200 2450 2000
-$Comp
 L Device:D_ALT D8
 U 1 1 5F685C97
@@
 Wire Wire Line
 	4250 2950 4250 3100
-Wire Wire Line
-	3200 2600 3200 2950
 $Comp
 L Connector:Conn_01x06_Male J16
@@
 $EndComp
 $Comp
-L Device:R R31
-U 1 1 5FBBFC18
-P 2700 2250
-F 0 "R31" H 2770 2296 50  0000 L CNN
-F 1 "100//100 5W (or 47ohm 7W)" H 2770 2205 50  0000 L CNN
-F 2 "Resistor_THT:R_Axial_DIN0617_L17.0mm_D6.0mm_P30.48mm_Horizontal" V 2630 2250 50  0001 C CNN
-F 3 "~" H 2700 2250 50  0001 C CNN
-	1    2700 2250
-	1    0    0    -1
-$EndComp
-$Comp
-L ossc_board-rescue:GND-RESCUE-ossc_board #PWR059
-U 1 1 5FBC0130
-P 2300 2650
-F 0 "#PWR059" H 2300 2650 30  0001 C CNN
-F 1 "GND-RESCUE-ossc_board" H 2300 2580 30  0001 C CNN
-F 2 "" H 2300 2650 60  0000 C CNN
-F 3 "" H 2300 2650 60  0000 C CNN
-	1    2300 2650
-	0    -1   -1   0
-$EndComp
-Wire Wire Line
-	2700 2100 2700 2000
-Wire Wire Line
-	2700 2000 2450 2000
-Connection ~ 2450 2000
-Wire Wire Line
-	2450 2000 2450 1850
-$Comp
 L ossc_board-rescue:FILTER FB?
 U 1 1 5FC17B44
@@
 P 3450 1650
 F 0 "#FLG0101" H 3450 1725 50  0001 C CNN
-F 1 "PWR_FLAG" H 3450 1823 50  0000 C CNN
+F 1 "PWR_FLAG" H 3450 1823 50  0001 C CNN
 F 2 "" H 3450 1650 50  0001 C CNN
 F 3 "~" H 3450 1650 50  0001 C CNN
@@
 P 3450 2850
 F 0 "#FLG0105" H 3450 2925 50  0001 C CNN
-F 1 "PWR_FLAG" H 3450 3023 50  0000 C CNN
+F 1 "PWR_FLAG" H 3450 3023 50  0001 C CNN
 F 2 "" H 3450 2850 50  0001 C CNN
 F 3 "~" H 3450 2850 50  0001 C CNN
@@
 	1    0    0    -1
 $EndComp
-Text Label 3200 2700 2    60   ~ 0
-5VDC_STBY
 Text Label 6800 7400 1    60   ~ 0
 VCCIO
@@
 	4900 1750 5050 1750
 Connection ~ 5050 1750
-Wire Wire Line
-	5050 2500 5050 1750
-Wire Wire Line
-	3200 2600 5050 2600
 $Comp
 L Connector_Generic:Conn_01x02 JP1
 U 1 1 5F692B96
-P 5250 2500
-F 0 "JP1" H 5330 2492 50  0000 L CNN
-F 1 "Standby DC From NeXT Hardware" H 5330 2401 50  0000 L CNN
-F 2 "Connector_PinHeader_2.54mm:PinHeader_1x02_P2.54mm_Vertical" H 5250 2500 50  0001 C CNN
-F 3 "~" H 5250 2500 50  0001 C CNN
-	1    5250 2500
+P 5550 2400
+F 0 "JP1" H 5630 2392 50  0000 L CNN
+F 1 "Standby DC From NeXT Hardware" H 4650 2200 50  0000 L CNN
+F 2 "Connector_PinHeader_2.54mm:PinHeader_1x02_P2.54mm_Vertical" H 5550 2400 50  0001 C CNN
+F 3 "~" H 5550 2400 50  0001 C CNN
+	1    5550 2400
 	1    0    0    -1
 $EndComp
-$Comp
-L Connector_Generic:Conn_01x02 JP6
-U 1 1 5F626198
-P 2100 2650
-F 0 "JP6" H 2180 2642 50  0000 L CNN
-F 1 "Use Dummy Load" H 2180 2551 50  0000 L CNN
-F 2 "Connector_PinHeader_2.54mm:PinHeader_1x02_P2.54mm_Vertical" H 2100 2650 50  0001 C CNN
-F 3 "~" H 2100 2650 50  0001 C CNN
-	1    2100 2650
-	-1   0    0    1
-$EndComp
-Wire Wire Line
-	2700 2400 2700 2550
-Wire Wire Line
-	2300 2550 2700 2550
 Wire Wire Line
 	11950 1100 11950 1450
@@
 $EndComp
 Wire Wire Line
-	5400 2200 5400 2300
-Wire Wire Line
-	5400 2300 4900 2300
-Connection ~ 4900 2300
-Wire Wire Line
 	5400 1800 5400 1650
 Wire Wire Line
@@
 Text Notes 2700 11050 0    60   ~ 0
 This block is optional.
-Text Notes 2750 2500 0    60   ~ 0
--12V Dummy Load for older PSU
+$Comp
+L Regulator_Linear:L7805 U33
+U 1 1 60E41152
+P 6350 2850
+F 0 "U33" H 6350 3092 50  0000 C CNN
+F 1 "5V(DC/DC)" H 6350 3001 50  0000 C CNN
+F 2 "Package_TO_SOT_THT:TO-220-3_Vertical" H 6375 2700 50  0001 L CIN
+F 3 "http://www.st.com/content/ccc/resource/technical/document/datasheet/41/4f/b3/b0/12/d4/47/88/CD00000444.pdf/files/CD00000444.pdf/jcr:content/translations/en.CD00000444.pdf" H 6350 2800 50  0001 C CNN
+	1    6350 2850
+	1    0    0    -1
+$EndComp
+$Comp
+L Device:C C181
+U 1 1 60E4115C
+P 6750 3100
+F 0 "C181" H 6865 3146 50  0000 L CNN
+F 1 "1u" H 6865 3055 50  0000 L CNN
+F 2 "Capacitor_SMD:C_0603_1608Metric_Pad1.08x0.95mm_HandSolder" H 6788 2950 50  0001 C CNN
+F 3 "~" H 6750 3100 50  0001 C CNN
+	1    6750 3100
+	1    0    0    1
+$EndComp
+Wire Wire Line
+	5650 2950 5650 2850
+Connection ~ 5650 2850
+Wire Wire Line
+	5650 2850 5350 2850
+Wire Wire Line
+	6650 2850 6750 2850
+Wire Wire Line
+	6750 2850 6750 2950
+Wire Wire Line
+	6750 3250 6750 3400
+Wire Wire Line
+	6750 3400 6350 3400
+Wire Wire Line
+	5650 3250 5650 3400
+Wire Wire Line
+	6350 3150 6350 3400
+Connection ~ 6350 3400
+Wire Wire Line
+	6350 3400 5950 3400
+Wire Wire Line
+	6350 3400 6350 3500
+Connection ~ 6750 2850
+$Comp
+L Device:CP C182
+U 1 1 60E41175
+P 7100 3100
+F 0 "C182" H 7218 3146 50  0000 L CNN
+F 1 "47u" H 7218 3055 50  0000 L CNN
+F 2 "Capacitor_SMD:CP_Elec_5x5.3" H 7138 2950 50  0001 C CNN
+F 3 "~" H 7100 3100 50  0001 C CNN
+	1    7100 3100
+	1    0    0    -1
+$EndComp
+Wire Wire Line
+	6750 2850 7100 2850
+Wire Wire Line
+	7100 2950 7100 2850
+Connection ~ 7100 2850
+Wire Wire Line
+	7100 3250 7100 3400
+Wire Wire Line
+	7100 3400 6750 3400
+Connection ~ 6750 3400
+$Comp
+L Device:C C179
+U 1 1 60E41185
+P 5650 3100
+F 0 "C179" H 5700 3000 50  0000 L CNN
+F 1 "1u" H 5750 3200 50  0000 L CNN
+F 2 "Capacitor_SMD:C_0603_1608Metric_Pad1.08x0.95mm_HandSolder" H 5688 2950 50  0001 C CNN
+F 3 "~" H 5650 3100 50  0001 C CNN
+	1    5650 3100
+	1    0    0    1
+$EndComp
+$Comp
+L Device:CP C180
+U 1 1 60E4118F
+P 5950 3100
+F 0 "C180" H 6068 3146 50  0000 L CNN
+F 1 "47u" H 6068 3055 50  0000 L CNN
+F 2 "Capacitor_SMD:CP_Elec_5x5.3" H 5988 2950 50  0001 C CNN
+F 3 "~" H 5950 3100 50  0001 C CNN
+	1    5950 3100
+	1    0    0    -1
+$EndComp
+Wire Wire Line
+	5650 2850 5950 2850
+Connection ~ 5950 2850
+Wire Wire Line
+	5950 2850 6050 2850
+Wire Wire Line
+	5950 3250 5950 3400
+Wire Wire Line
+	5950 3400 5650 3400
+Connection ~ 5950 3400
+$Comp
+L power:PWR_FLAG #FLG01
+U 1 1 60E411A0
+P 5650 2750
+F 0 "#FLG01" H 5650 2825 50  0001 C CNN
+F 1 "PWR_FLAG" H 5650 2923 50  0001 C CNN
+F 2 "" H 5650 2750 50  0001 C CNN
+F 3 "~" H 5650 2750 50  0001 C CNN
+	1    5650 2750
+	1    0    0    -1
+$EndComp
+Wire Wire Line
+	5650 2750 5650 2850
+Wire Wire Line
+	5950 2850 5950 2950
+Wire Wire Line
+	6200 2450 5950 2450
+Wire Wire Line
+	5950 2450 5950 2850
+Wire Wire Line
+	6500 2450 6750 2450
+Wire Wire Line
+	6750 2450 6750 2850
+$Comp
+L Device:D_ALT D12
+U 1 1 60E411B0
+P 6350 2450
+F 0 "D12" V 6304 2529 50  0000 L CNN
+F 1 "(RB160M-30TR)" V 6450 2500 50  0000 L CNN
+F 2 "custom_components:D_SOD-123_HandSoldering" H 6350 2450 50  0001 C CNN
+F 3 "~" H 6350 2450 50  0001 C CNN
+	1    6350 2450
+	1    0    0    -1
+$EndComp
+Wire Wire Line
+	7100 2850 7250 2850
+Text Label 3200 2600 2    60   ~ 0
+5VDC_STBY
+Wire Wire Line
+	3200 2600 3200 2950
+Text Label 7250 2850 0    60   ~ 0
+5VDC_STBY
+$Comp
+L ossc_board-rescue:GND-RESCUE-ossc_board #PWR0274
+U 1 1 6134DCC1
+P 6350 3500
+F 0 "#PWR0274" H 6350 3500 30  0001 C CNN
+F 1 "GND-RESCUE-ossc_board" H 6350 3430 30  0001 C CNN
+F 2 "" H 6350 3500 60  0000 C CNN
+F 3 "" H 6350 3500 60  0000 C CNN
+	1    6350 3500
+	1    0    0    -1
+$EndComp
+Wire Wire Line
+	5350 2500 5350 2850
+NoConn ~ 1800 1850
+NoConn ~ 2200 1850
+Text Notes 1950 2000 0    60   ~ 0
+-12V not used
+Wire Wire Line
+	5400 2200 5400 2300
+Connection ~ 4900 2300
+Wire Wire Line
+	5400 2300 4900 2300
+Wire Wire Line
+	5350 2400 4450 2400
+Wire Wire Line
+	4450 2400 4450 2500
+Wire Wire Line
+	4450 2500 3300 2500
+Wire Wire Line
+	3300 2500 3300 1750
+Connection ~ 3300 1750
+Wire Wire Line
+	3300 1750 3150 1750
 $EndSCHEMATC

Commit message: update values
Parts:
- C172: value 0.1u -> 0.1u (GCJ188R71H104KA12D or GRM188R72A104MA35D)
- Y2: value 25MHz (FA-238 25.0000MB-K0) -> 25MHz (FA-238 25.0000MB-K0 or NX3225GA-25.000M-STD-CRG)
Other:
- note added: "auc. xxxA"
- note added: "max. 0mA"
- note added: "max. 2mA"
- note added: "max. 40mA@0.1W"
- note added: "max. 4mA"
- note added: "max. DAC+ADC=17mA"
- note added: "max. DAC+ADC=36mA"
- note removed: "max. DAC+ADC="
Changed lines of the file:
@@
 max. 32mA
 Text Notes 6450 750  0    60   ~ 0
-max. DAC+ADC=
+max. DAC+ADC=17mA
 Text Notes 8050 750  0    60   ~ 0
-max. DAC+ADC=
+max. DAC+ADC=36mA
 Text Notes 4200 2800 0    60   ~ 0
 max. MCU=
@@
 P 8700 6000
 F 0 "Y2" V 8654 6244 50  0000 L CNN
-F 1 "25MHz (FA-238 25.0000MB-K0)" V 8450 5250 50  0000 L CNN
+F 1 "25MHz (FA-238 25.0000MB-K0 or NX3225GA-25.000M-STD-CRG)" H 6900 5450 50  0000 L CNN
 F 2 "Crystal:Crystal_SMD_SeikoEpson_TSX3225-4Pin_3.2x2.5mm_HandSoldering" H 8700 6000 50  0001 C CNN
 F 3 "~" H 8700 6000 50  0001 C CNN
@@
 P 8800 4150
 F 0 "C172" H 8915 4196 50  0000 L CNN
-F 1 "0.1u" H 8915 4105 50  0000 L CNN
+F 1 "0.1u (GCJ188R71H104KA12D or GRM188R72A104MA35D)" H 8550 4500 50  0000 L CNN
 F 2 "Capacitor_SMD:C_0603_1608Metric_Pad1.05x0.95mm_HandSolder" H 8838 4000 50  0001 C CNN
 F 3 "~" H 8800 4150 50  0001 C CNN
@@
 Wire Wire Line
 	3300 1750 3150 1750
+Text Notes 3250 1450 0    60   ~ 0
+auc. xxxA
+Text Notes 5400 2800 0    60   ~ 0
+auc. xxxA
+Text Notes 6000 8400 0    60   ~ 0
+max. 4mA
+Text Notes 7250 8050 0    60   ~ 0
+max. 0mA
+Text Notes 7750 8450 0    60   ~ 0
+max. 2mA
+Text Notes 15550 3150 0    60   ~ 0
+max. 40mA@0.1W
 $EndSCHEMATC

Commit message: update
Parts:
- U33: value 5V(DC/DC) -> 5V(DC/DC) 0.7A max
- U8: value 5V(DC/DC) -> 5V(DC/DC) 1A(+0.1A D class amp) max
Other:
- note added: "max. 80mA@0.1W@4Ω"
- note removed: "max. 40mA@0.1W"
Changed lines of the file:
@@
 P 4150 1750
 F 0 "U8" H 4150 1992 50  0000 C CNN
-F 1 "5V(DC/DC)" H 4150 1901 50  0000 C CNN
+F 1 "5V(DC/DC) 1A(+0.1A D class amp) max" H 4150 1901 50  0000 C CNN
 F 2 "Package_TO_SOT_THT:TO-220-3_Vertical" H 4175 1600 50  0001 L CIN
 F 3 "http://www.st.com/content/ccc/resource/technical/document/datasheet/41/4f/b3/b0/12/d4/47/88/CD00000444.pdf/files/CD00000444.pdf/jcr:content/translations/en.CD00000444.pdf" H 4150 1700 50  0001 C CNN
@@
 P 6350 2850
 F 0 "U33" H 6350 3092 50  0000 C CNN
-F 1 "5V(DC/DC)" H 6350 3001 50  0000 C CNN
+F 1 "5V(DC/DC) 0.7A max" H 6350 3001 50  0000 C CNN
 F 2 "Package_TO_SOT_THT:TO-220-3_Vertical" H 6375 2700 50  0001 L CIN
 F 3 "http://www.st.com/content/ccc/resource/technical/document/datasheet/41/4f/b3/b0/12/d4/47/88/CD00000444.pdf/files/CD00000444.pdf/jcr:content/translations/en.CD00000444.pdf" H 6350 2800 50  0001 C CNN
@@
 max. 2mA
 Text Notes 15550 3150 0    60   ~ 0
-max. 40mA@0.1W
+max. 80mA@0.1W@4Ω
 $EndSCHEMATC
